File: template/Hammond_1598A/1598A.kicad_pcb (KiCad board)
At the start: 2 copper layers, 0 parts

Commit message: feat: Add Templates for Hammond Enclosures
create template for 1598A

Issue #17
Parts:
- added ~: ~, MountingHole:MountingHole_3.5mm_Pad, F.Cu at (27.3, 80.2)
- added ~: ~, MountingHole:MountingHole_3.5mm_Pad, F.Cu at (27.3, 29.8)
- added ~: ~, MountingHole:MountingHole_3.5mm_Pad, F.Cu at (147.3, 80.2)
- added ~: ~, MountingHole:MountingHole_3.5mm_Pad, F.Cu at (147.3, 29.8)
Other:
- board outline added: 144.6 x 80 mm
Changed lines of the file:
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@@
   (general
     (thickness 1.6)
-    (drawings 0)
+    (drawings 14)
     (tracks 0)
     (zones 0)
-    (modules 0)
+    (modules 4)
     (nets 1)
   )
@@
     (pad_to_mask_clearance 0.051)
     (solder_mask_min_width 0.25)
-    (aux_axis_origin 15 44.5)
+    (aux_axis_origin 15 95)
     (visible_elements 7FFFFFFF)
     (pcbplotparams
@@
     (uvia_drill 0.1)
   )
+  (module MountingHole:MountingHole_3.5mm_Pad (layer F.Cu)
+    (at 27.3 80.19)
+    (descr "Mounting Hole 3.5mm")
+    (tags "mounting hole 3.5mm")
+    (attr virtual)
+    (fp_text reference ~ (at 0 -4.5) (layer F.SilkS) hide
+      (effects (font (size 1 1) (thickness 0.15)))
+    )
+    (fp_text value ~ (at 0 4.5) (layer F.Fab) hide
+      (effects (font (size 1 1) (thickness 0.15)))
+    )
+    (fp_text user %R (at 0.3 0) (layer F.Fab)
+      (effects (font (size 1 1) (thickness 0.15)))
+    )
+    (fp_circle (center 0 0) (end 3.5 0) (layer Cmts.User) (width 0.15))
+    (fp_circle (center 0 0) (end 3.75 0) (layer F.CrtYd) (width 0.05))
+    (pad 1 thru_hole circle (at 0 0) (size 7 7) (drill 3.5) (layers *.Cu *.Mask))
+  )
+  (module MountingHole:MountingHole_3.5mm_Pad (layer F.Cu)
+    (at 27.3 29.81)
+    (descr "Mounting Hole 3.5mm")
+    (tags "mounting hole 3.5mm")
+    (attr virtual)
+    (fp_text reference ~ (at 0 -4.5) (layer F.SilkS) hide
+      (effects (font (size 1 1) (thickness 0.15)))
+    )
+    (fp_text value ~ (at 0 4.5) (layer F.Fab) hide
+      (effects (font (size 1 1) (thickness 0.15)))
+    )
+    (fp_circle (center 0 0) (end 3.75 0) (layer F.CrtYd) (width 0.05))
+    (fp_circle (center 0 0) (end 3.5 0) (layer Cmts.User) (width 0.15))
+    (fp_text user %R (at 0.3 0) (layer F.Fab)
+      (effects (font (size 1 1) (thickness 0.15)))
+    )
+    (pad 1 thru_hole circle (at 0 0) (size 7 7) (drill 3.5) (layers *.Cu *.Mask))
+  )
+  (module MountingHole:MountingHole_3.5mm_Pad (layer F.Cu)
+    (at 147.3 80.19)
+    (descr "Mounting Hole 3.5mm")
+    (tags "mounting hole 3.5mm")
+    (attr virtual)
+    (fp_text reference ~ (at 0 -4.5) (layer F.SilkS) hide
+      (effects (font (size 1 1) (thickness 0.15)))
+    )
+    (fp_text value ~ (at 0 4.5) (layer F.Fab) hide
+      (effects (font (size 1 1) (thickness 0.15)))
+    )
+    (fp_text user %R (at 0.3 0) (layer F.Fab)
+      (effects (font (size 1 1) (thickness 0.15)))
+    )
+    (fp_circle (center 0 0) (end 3.5 0) (layer Cmts.User) (width 0.15))
+    (fp_circle (center 0 0) (end 3.75 0) (layer F.CrtYd) (width 0.05))
+    (pad 1 thru_hole circle (at 0 0) (size 7 7) (drill 3.5) (layers *.Cu *.Mask))
+  )
+  (module MountingHole:MountingHole_3.5mm_Pad (layer F.Cu)
+    (at 147.3 29.81)
+    (descr "Mounting Hole 3.5mm")
+    (tags "mounting hole 3.5mm")
+    (attr virtual)
+    (fp_text reference ~ (at 0 -4.5) (layer F.SilkS) hide
+      (effects (font (size 1 1) (thickness 0.15)))
+    )
+    (fp_text value ~ (at 0 4.5) (layer F.Fab) hide
+      (effects (font (size 1 1) (thickness 0.15)))
+    )
+    (fp_circle (center 0 0) (end 3.75 0) (layer F.CrtYd) (width 0.05))
+    (fp_circle (center 0 0) (end 3.5 0) (layer Cmts.User) (width 0.15))
+    (fp_text user %R (at 0.3 0) (layer F.Fab)
+      (effects (font (size 1 1) (thickness 0.15)))
+    )
+    (pad 1 thru_hole circle (at 0 0) (size 7 7) (drill 3.5) (layers *.Cu *.Mask))
+  )
+  (dimension 80 (width 0.15) (layer Dwgs.User)
+    (gr_text "80,000 mm" (at 165.9 55 90) (layer Dwgs.User)
+      (effects (font (size 1 1) (thickness 0.15)))
+    )
+    (feature1 (pts (xy 159.6 15) (xy 165.186421 15)))
+    (feature2 (pts (xy 159.6 95) (xy 165.186421 95)))
+    (crossbar (pts (xy 164.6 95) (xy 164.6 15)))
+    (arrow1a (pts (xy 164.6 15) (xy 165.186421 16.126504)))
+    (arrow1b (pts (xy 164.6 15) (xy 164.013579 16.126504)))
+    (arrow2a (pts (xy 164.6 95) (xy 165.186421 93.873496)))
+    (arrow2b (pts (xy 164.6 95) (xy 164.013579 93.873496)))
+  )
+  (dimension 144.6 (width 0.15) (layer Dwgs.User)
+    (gr_text "144,600 mm" (at 87.3 101.3) (layer Dwgs.User)
+      (effects (font (size 1 1) (thickness 0.15)))
+    )
+    (feature1 (pts (xy 159.6 95) (xy 159.6 100.586421)))
+    (feature2 (pts (xy 15 95) (xy 15 100.586421)))
+    (crossbar (pts (xy 15 100) (xy 159.6 100)))
+    (arrow1a (pts (xy 159.6 100) (xy 158.473496 100.586421)))
+    (arrow1b (pts (xy 159.6 100) (xy 158.473496 99.413579)))
+    (arrow2a (pts (xy 15 100) (xy 16.126504 100.586421)))
+    (arrow2b (pts (xy 15 100) (xy 16.126504 99.413579)))
+  )
+  (gr_line (start 93.5 95) (end 159.6 95) (layer Edge.Cuts) (width 0.05))
+  (gr_arc (start 87.3 90.65) (end 93.5 90.65) (angle -180) (layer Edge.Cuts) (width 0.05))
+  (gr_line (start 93.5 90.65) (end 93.5 95) (layer Edge.Cuts) (width 0.05))
+  (gr_line (start 81.1 90.65) (end 81.1 95) (layer Edge.Cuts) (width 0.05))
+  (gr_line (start 93.5 15) (end 159.6 15) (layer Edge.Cuts) (width 0.05))
+  (gr_arc (start 87.3 19.35) (end 81.1 19.35) (angle -180) (layer Edge.Cuts) (width 0.05))
+  (gr_line (start 81.1 15) (end 81.1 19.35) (layer Edge.Cuts) (width 0.05))
+  (gr_line (start 93.5 15) (end 93.5 19.35) (layer Edge.Cuts) (width 0.05))
+  (gr_line (start 159.6 95) (end 159.6 15) (layer Edge.Cuts) (width 0.05))
+  (gr_line (start 15 15) (end 15 95) (layer Edge.Cuts) (width 0.05))
+  (gr_line (start 15 95) (end 81.1 95) (layer Edge.Cuts) (width 0.05))
+  (gr_line (start 15 15) (end 81.1 15) (layer Edge.Cuts) (width 0.05))
 )
