File: template/Hammond_1598B/1598B.kicad_pcb (KiCad board)
At the start: 2 copper layers, 0 parts

Commit message: feat: Add Templates for Hammond Enclosures
fix bugs, add board images

Issue #17
Parts:
- added ~: ~, MountingHole:MountingHole_3.5mm_Pad, F.Cu at (44.0, 114.2)
- added ~: ~, MountingHole:MountingHole_3.5mm_Pad, F.Cu at (44.0, 37.8)
- added ~: ~, MountingHole:MountingHole_3.5mm_Pad, F.Cu at (108.3, 114.2)
- added ~: ~, MountingHole:MountingHole_3.5mm_Pad, F.Cu at (108.3, 37.8)
- added ~: ~, MountingHole:MountingHole_3.5mm_Pad, F.Cu at (76.2, 114.2)
- added ~: ~, MountingHole:MountingHole_3.5mm_Pad, F.Cu at (76.2, 37.8)
Other:
- board outline added: 122.3 x 122 mm
Changed lines of the file:
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@@
   (general
     (thickness 1.6)
-    (drawings 0)
+    (drawings 14)
     (tracks 0)
     (zones 0)
-    (modules 0)
+    (modules 6)
     (nets 1)
   )
@@
     (mod_text_size 1 1)
     (mod_text_width 0.15)
-    (pad_size 1.524 1.524)
-    (pad_drill 0.762)
+    (pad_size 7 7)
+    (pad_drill 3.5)
     (pad_to_mask_clearance 0.051)
     (solder_mask_min_width 0.25)
-    (aux_axis_origin 15 44.5)
+    (aux_axis_origin 15 137)
     (visible_elements 7FFFFFFF)
     (pcbplotparams
@@
     (uvia_drill 0.1)
   )
+  (module MountingHole:MountingHole_3.5mm_Pad (layer F.Cu)
+    (at 44 114.2)
+    (descr "Mounting Hole 3.5mm")
+    (tags "mounting hole 3.5mm")
+    (attr virtual)
+    (fp_text reference ~ (at 0 -4.5) (layer F.SilkS) hide
+      (effects (font (size 1 1) (thickness 0.15)))
+    )
+    (fp_text value ~ (at 0 4.5) (layer F.Fab) hide
+      (effects (font (size 1 1) (thickness 0.15)))
+    )
+    (fp_text user %R (at 0.3 0) (layer F.Fab)
+      (effects (font (size 1 1) (thickness 0.15)))
+    )
+    (fp_circle (center 0 0) (end 3.5 0) (layer Cmts.User) (width 0.15))
+    (fp_circle (center 0 0) (end 3.75 0) (layer F.CrtYd) (width 0.05))
+    (pad ~ thru_hole circle (at 0 0) (size 7 7) (drill 3.5) (layers *.Cu *.Mask))
+  )
+  (module MountingHole:MountingHole_3.5mm_Pad (layer F.Cu)
+    (at 44 37.8)
+    (descr "Mounting Hole 3.5mm")
+    (tags "mounting hole 3.5mm")
+    (attr virtual)
+    (fp_text reference ~ (at 0 -4.5) (layer F.SilkS) hide
+      (effects (font (size 1 1) (thickness 0.15)))
+    )
+    (fp_text value ~ (at 0 4.5) (layer F.Fab) hide
+      (effects (font (size 1 1) (thickness 0.15)))
+    )
+    (fp_text user %R (at 0.3 0) (layer F.Fab)
+      (effects (font (size 1 1) (thickness 0.15)))
+    )
+    (fp_circle (center 0 0) (end 3.5 0) (layer Cmts.User) (width 0.15))
+    (fp_circle (center 0 0) (end 3.75 0) (layer F.CrtYd) (width 0.05))
+    (pad ~ thru_hole circle (at 0 0) (size 7 7) (drill 3.5) (layers *.Cu *.Mask))
+  )
+  (module MountingHole:MountingHole_3.5mm_Pad (layer F.Cu)
+    (at 108.3 114.2)
+    (descr "Mounting Hole 3.5mm")
+    (tags "mounting hole 3.5mm")
+    (attr virtual)
+    (fp_text reference ~ (at 0 -4.5) (layer F.SilkS) hide
+      (effects (font (size 1 1) (thickness 0.15)))
+    )
+    (fp_text value ~ (at 0 4.5) (layer F.Fab) hide
+      (effects (font (size 1 1) (thickness 0.15)))
+    )
+    (fp_text user %R (at 0.3 0) (layer F.Fab)
+      (effects (font (size 1 1) (thickness 0.15)))
+    )
+    (fp_circle (center 0 0) (end 3.5 0) (layer Cmts.User) (width 0.15))
+    (fp_circle (center 0 0) (end 3.75 0) (layer F.CrtYd) (width 0.05))
+    (pad ~ thru_hole circle (at 0 0) (size 7 7) (drill 3.5) (layers *.Cu *.Mask))
+  )
+  (module MountingHole:MountingHole_3.5mm_Pad (layer F.Cu)
+    (at 108.3 37.8)
+    (descr "Mounting Hole 3.5mm")
+    (tags "mounting hole 3.5mm")
+    (attr virtual)
+    (fp_text reference ~ (at 0 -4.5) (layer F.SilkS) hide
+      (effects (font (size 1 1) (thickness 0.15)))
+    )
+    (fp_text value ~ (at 0 4.5) (layer F.Fab) hide
+      (effects (font (size 1 1) (thickness 0.15)))
+    )
+    (fp_circle (center 0 0) (end 3.75 0) (layer F.CrtYd) (width 0.05))
+    (fp_circle (center 0 0) (end 3.5 0) (layer Cmts.User) (width 0.15))
+    (fp_text user %R (at 0.3 0) (layer F.Fab)
+      (effects (font (size 1 1) (thickness 0.15)))
+    )
+    (pad ~ thru_hole circle (at 0 0) (size 7 7) (drill 3.5) (layers *.Cu *.Mask))
+  )
+  (module MountingHole:MountingHole_3.5mm_Pad (layer F.Cu)
+    (at 76.15 114.2)
+    (descr "Mounting Hole 3.5mm")
+    (tags "mounting hole 3.5mm")
+    (attr virtual)
+    (fp_text reference ~ (at 0 -4.5) (layer F.SilkS) hide
+      (effects (font (size 1 1) (thickness 0.15)))
+    )
+    (fp_text value ~ (at 0 4.5) (layer F.Fab) hide
+      (effects (font (size 1 1) (thickness 0.15)))
+    )
+    (fp_text user %R (at 0.3 0) (layer F.Fab)
+      (effects (font (size 1 1) (thickness 0.15)))
+    )
+    (fp_circle (center 0 0) (end 3.5 0) (layer Cmts.User) (width 0.15))
+    (fp_circle (center 0 0) (end 3.75 0) (layer F.CrtYd) (width 0.05))
+    (pad ~ thru_hole circle (at 0 0) (size 7 7) (drill 3.5) (layers *.Cu *.Mask))
+  )
+  (module MountingHole:MountingHole_3.5mm_Pad (layer F.Cu)
+    (at 76.15 37.8)
+    (descr "Mounting Hole 3.5mm")
+    (tags "mounting hole 3.5mm")
+    (attr virtual)
+    (fp_text reference ~ (at 0 -4.5) (layer F.SilkS) hide
+      (effects (font (size 1 1) (thickness 0.15)))
+    )
+    (fp_text value ~ (at 0 4.5) (layer F.Fab) hide
+      (effects (font (size 1 1) (thickness 0.15)))
+    )
+    (fp_circle (center 0 0) (end 3.75 0) (layer F.CrtYd) (width 0.05))
+    (fp_circle (center 0 0) (end 3.5 0) (layer Cmts.User) (width 0.15))
+    (fp_text user %R (at 0.3 0) (layer F.Fab)
+      (effects (font (size 1 1) (thickness 0.15)))
+    )
+    (pad ~ thru_hole circle (at 0 0) (size 7 7) (drill 3.5) (layers *.Cu *.Mask))
+  )
+  (gr_line (start 82.35 137) (end 137.3 137) (layer Edge.Cuts) (width 0.05))
+  (gr_arc (start 76.15 132.67) (end 82.35 132.67) (angle -180) (layer Edge.Cuts) (width 0.05))
+  (gr_line (start 82.35 132.67) (end 82.35 137) (layer Edge.Cuts) (width 0.05))
+  (gr_line (start 69.95 132.67) (end 69.95 137) (layer Edge.Cuts) (width 0.05))
+  (gr_arc (start 76.15 19.33) (end 69.95 19.33) (angle -180) (layer Edge.Cuts) (width 0.05))
+  (gr_line (start 82.35 15) (end 137.3 15) (layer Edge.Cuts) (width 0.05))
+  (gr_line (start 69.95 15) (end 69.95 19.33) (layer Edge.Cuts) (width 0.05))
+  (gr_line (start 82.35 15) (end 82.35 19.33) (layer Edge.Cuts) (width 0.05))
+  (dimension 122 (width 0.15) (layer Dwgs.User)
+    (gr_text "122,000 mm" (at 143.6 76 90) (layer Dwgs.User)
+      (effects (font (size 1 1) (thickness 0.15)))
+    )
+    (feature1 (pts (xy 137.3 15) (xy 142.886421 15)))
+    (feature2 (pts (xy 137.3 137) (xy 142.886421 137)))
+    (crossbar (pts (xy 142.3 137) (xy 142.3 15)))
+    (arrow1a (pts (xy 142.3 15) (xy 142.886421 16.126504)))
+    (arrow1b (pts (xy 142.3 15) (xy 141.713579 16.126504)))
+    (arrow2a (pts (xy 142.3 137) (xy 142.886421 135.873496)))
+    (arrow2b (pts (xy 142.3 137) (xy 141.713579 135.873496)))
+  )
+  (dimension 122.3 (width 0.15) (layer Dwgs.User)
+    (gr_text "122,300 mm" (at 76.15 143.3) (layer Dwgs.User)
+      (effects (font (size 1 1) (thickness 0.15)))
+    )
+    (feature1 (pts (xy 137.3 137) (xy 137.3 142.586421)))
+    (feature2 (pts (xy 15 137) (xy 15 142.586421)))
+    (crossbar (pts (xy 15 142) (xy 137.3 142)))
+    (arrow1a (pts (xy 137.3 142) (xy 136.173496 142.586421)))
+    (arrow1b (pts (xy 137.3 142) (xy 136.173496 141.413579)))
+    (arrow2a (pts (xy 15 142) (xy 16.126504 142.586421)))
+    (arrow2b (pts (xy 15 142) (xy 16.126504 141.413579)))
+  )
+  (gr_line (start 137.3 137) (end 137.3 15) (layer Edge.Cuts) (width 0.05))
+  (gr_line (start 15 15) (end 15 137) (layer Edge.Cuts) (width 0.05))
+  (gr_line (start 15 137) (end 69.95 137) (layer Edge.Cuts) (width 0.05))
+  (gr_line (start 15 15) (end 69.95 15) (layer Edge.Cuts) (width 0.05))
 )
