File: template/Hammond_1598BB/1598BB.kicad_pcb (KiCad board)
At the start: 2 copper layers, 0 parts

Commit message: feat: Add Templates for Hammond Enclosures
fix bugs, add board images

Issue #17
Parts:
- added ~: ~, MountingHole:MountingHole_3.5mm_Pad, F.Cu at (26.6, 38.3)
- added ~: ~, MountingHole:MountingHole_3.5mm_Pad, F.Cu at (26.6, 132.7)
- added ~: ~, MountingHole:MountingHole_3.5mm_Pad, F.Cu at (171.2, 38.3)
- added ~: ~, MountingHole:MountingHole_3.5mm_Pad, F.Cu at (171.2, 132.7)
Other:
- board outline added: 167.8 x 141 mm
Changed lines of the file:
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@@
   (general
     (thickness 1.6)
-    (drawings 0)
+    (drawings 14)
     (tracks 0)
     (zones 0)
-    (modules 0)
+    (modules 4)
     (nets 1)
   )
@@
     (mod_text_size 1 1)
     (mod_text_width 0.15)
-    (pad_size 1.524 1.524)
-    (pad_drill 0.762)
+    (pad_size 7 7)
+    (pad_drill 3.5)
     (pad_to_mask_clearance 0.051)
     (solder_mask_min_width 0.25)
-    (aux_axis_origin 15 44.5)
+    (aux_axis_origin 15 156)
     (visible_elements 7FFFFFFF)
     (pcbplotparams
@@
     (uvia_drill 0.1)
   )
+  (module MountingHole:MountingHole_3.5mm_Pad (layer F.Cu)
+    (at 26.58 38.3)
+    (descr "Mounting Hole 3.5mm")
+    (tags "mounting hole 3.5mm")
+    (attr virtual)
+    (fp_text reference ~ (at 0 -4.5) (layer F.SilkS) hide
+      (effects (font (size 1 1) (thickness 0.15)))
+    )
+    (fp_text value ~ (at 0 4.5) (layer F.Fab) hide
+      (effects (font (size 1 1) (thickness 0.15)))
+    )
+    (fp_text user %R (at 0.3 0) (layer F.Fab)
+      (effects (font (size 1 1) (thickness 0.15)))
+    )
+    (fp_circle (center 0 0) (end 3.5 0) (layer Cmts.User) (width 0.15))
+    (fp_circle (center 0 0) (end 3.75 0) (layer F.CrtYd) (width 0.05))
+    (pad ~ thru_hole circle (at 0 0) (size 7 7) (drill 3.5) (layers *.Cu *.Mask))
+  )
+  (module MountingHole:MountingHole_3.5mm_Pad (layer F.Cu)
+    (at 26.58 132.7)
+    (descr "Mounting Hole 3.5mm")
+    (tags "mounting hole 3.5mm")
+    (attr virtual)
+    (fp_text reference ~ (at 0 -4.5) (layer F.SilkS) hide
+      (effects (font (size 1 1) (thickness 0.15)))
+    )
+    (fp_text value ~ (at 0 4.5) (layer F.Fab) hide
+      (effects (font (size 1 1) (thickness 0.15)))
+    )
+    (fp_circle (center 0 0) (end 3.75 0) (layer F.CrtYd) (width 0.05))
+    (fp_circle (center 0 0) (end 3.5 0) (layer Cmts.User) (width 0.15))
+    (fp_text user %R (at 0.3 0) (layer F.Fab)
+      (effects (font (size 1 1) (thickness 0.15)))
+    )
+    (pad ~ thru_hole circle (at 0 0) (size 7 7) (drill 3.5) (layers *.Cu *.Mask))
+  )
+  (module MountingHole:MountingHole_3.5mm_Pad (layer F.Cu)
+    (at 171.22 38.3)
+    (descr "Mounting Hole 3.5mm")
+    (tags "mounting hole 3.5mm")
+    (attr virtual)
+    (fp_text reference ~ (at 0 -4.5) (layer F.SilkS) hide
+      (effects (font (size 1 1) (thickness 0.15)))
+    )
+    (fp_text value ~ (at 0 4.5) (layer F.Fab) hide
+      (effects (font (size 1 1) (thickness 0.15)))
+    )
+    (fp_text user %R (at 0.3 0) (layer F.Fab)
+      (effects (font (size 1 1) (thickness 0.15)))
+    )
+    (fp_circle (center 0 0) (end 3.5 0) (layer Cmts.User) (width 0.15))
+    (fp_circle (center 0 0) (end 3.75 0) (layer F.CrtYd) (width 0.05))
+    (pad ~ thru_hole circle (at 0 0) (size 7 7) (drill 3.5) (layers *.Cu *.Mask))
+  )
+  (module MountingHole:MountingHole_3.5mm_Pad (layer F.Cu)
+    (at 171.22 132.7)
+    (descr "Mounting Hole 3.5mm")
+    (tags "mounting hole 3.5mm")
+    (attr virtual)
+    (fp_text reference ~ (at 0 -4.5) (layer F.SilkS) hide
+      (effects (font (size 1 1) (thickness 0.15)))
+    )
+    (fp_text value ~ (at 0 4.5) (layer F.Fab) hide
+      (effects (font (size 1 1) (thickness 0.15)))
+    )
+    (fp_circle (center 0 0) (end 3.75 0) (layer F.CrtYd) (width 0.05))
+    (fp_circle (center 0 0) (end 3.5 0) (layer Cmts.User) (width 0.15))
+    (fp_text user %R (at 0.3 0) (layer F.Fab)
+      (effects (font (size 1 1) (thickness 0.15)))
+    )
+    (pad ~ thru_hole circle (at 0 0) (size 7 7) (drill 3.5) (layers *.Cu *.Mask))
+  )
+  (gr_line (start 105.1 156) (end 182.8 156) (layer Edge.Cuts) (width 0.05))
+  (gr_arc (start 98.9 151.2) (end 105.1 151.2) (angle -180) (layer Edge.Cuts) (width 0.05))
+  (gr_line (start 92.7 151.2) (end 92.7 156) (layer Edge.Cuts) (width 0.05))
+  (gr_line (start 105.1 151.2) (end 105.1 156) (layer Edge.Cuts) (width 0.05))
+  (gr_line (start 105.1 15) (end 182.8 15) (layer Edge.Cuts) (width 0.05))
+  (gr_arc (start 98.9 19.8) (end 92.7 19.8) (angle -180) (layer Edge.Cuts) (width 0.05))
+  (gr_line (start 92.7 15) (end 92.7 19.8) (layer Edge.Cuts) (width 0.05))
+  (gr_line (start 105.1 15) (end 105.1 19.8) (layer Edge.Cuts) (width 0.05))
+  (dimension 141 (width 0.15) (layer Dwgs.User)
+    (gr_text "141,000 mm" (at 189.3 85.5 90) (layer Dwgs.User)
+      (effects (font (size 1 1) (thickness 0.15)))
+    )
+    (feature1 (pts (xy 182.8 15) (xy 188.586421 15)))
+    (feature2 (pts (xy 182.8 156) (xy 188.586421 156)))
+    (crossbar (pts (xy 188 156) (xy 188 15)))
+    (arrow1a (pts (xy 188 15) (xy 188.586421 16.126504)))
+    (arrow1b (pts (xy 188 15) (xy 187.413579 16.126504)))
+    (arrow2a (pts (xy 188 156) (xy 188.586421 154.873496)))
+    (arrow2b (pts (xy 188 156) (xy 187.413579 154.873496)))
+  )
+  (dimension 167.8 (width 0.15) (layer Dwgs.User)
+    (gr_text "167,800 mm" (at 98.9 162.3) (layer Dwgs.User)
+      (effects (font (size 1 1) (thickness 0.15)))
+    )
+    (feature1 (pts (xy 182.8 156) (xy 182.8 161.586421)))
+    (feature2 (pts (xy 15 156) (xy 15 161.586421)))
+    (crossbar (pts (xy 15 161) (xy 182.8 161)))
+    (arrow1a (pts (xy 182.8 161) (xy 181.673496 161.586421)))
+    (arrow1b (pts (xy 182.8 161) (xy 181.673496 160.413579)))
+    (arrow2a (pts (xy 15 161) (xy 16.126504 161.586421)))
+    (arrow2b (pts (xy 15 161) (xy 16.126504 160.413579)))
+  )
+  (gr_line (start 182.8 156) (end 182.8 15) (layer Edge.Cuts) (width 0.05))
+  (gr_line (start 15 15) (end 15 156) (layer Edge.Cuts) (width 0.05))
+  (gr_line (start 15 156) (end 92.7 156) (layer Edge.Cuts) (width 0.05))
+  (gr_line (start 15 15) (end 92.7 15) (layer Edge.Cuts) (width 0.05))
 )
