File: template/Hammond_RM2015L/RM2015L.kicad_pcb (KiCad board)
At the start: 2 copper layers, 123 x 88 mm, 4 parts

Commit message: feat: Add Templates for Hammond Enclosures
fix mounting hole pad number

Issue #17
Parts:
- ~ (x4): renamed from REF**; value MountingHole_3.5mm_Pad -> ~
Changed lines of the file:
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@@
     (mod_text_size 1 1)
     (mod_text_width 0.15)
-    (pad_size 1.524 1.524)
-    (pad_drill 0.762)
+    (pad_size 7 7)
+    (pad_drill 3.5)
     (pad_to_mask_clearance 0.051)
     (solder_mask_min_width 0.25)
-    (aux_axis_origin 0 0)
-    (visible_elements FFFFFF7F)
+    (aux_axis_origin 15 103)
+    (visible_elements 7FFFFFFF)
     (pcbplotparams
       (layerselection 0x010fc_ffffffff)
@@
     (tags "mounting hole 3.5mm")
     (attr virtual)
-    (fp_text reference REF** (at 0 -4.5) (layer F.SilkS) hide
+    (fp_text reference ~ (at 0 -4.5) (layer F.SilkS) hide
       (effects (font (size 1 1) (thickness 0.15)))
     )
-    (fp_text value MountingHole_3.5mm_Pad (at 0 4.5) (layer F.Fab) hide
+    (fp_text value ~ (at 0 4.5) (layer F.Fab) hide
       (effects (font (size 1 1) (thickness 0.15)))
     )
@@
     (fp_circle (center 0 0) (end 3.5 0) (layer Cmts.User) (width 0.15))
     (fp_circle (center 0 0) (end 3.75 0) (layer F.CrtYd) (width 0.05))
-    (pad 1 thru_hole circle (at 0 0) (size 7 7) (drill 3.5) (layers *.Cu *.Mask))
+    (pad ~ thru_hole circle (at 0 0) (size 7 7) (drill 3.5) (layers *.Cu *.Mask))
   )
   (module MountingHole:MountingHole_3.5mm_Pad (layer F.Cu)
@@
     (tags "mounting hole 3.5mm")
     (attr virtual)
-    (fp_text reference REF** (at 0 -4.5) (layer F.SilkS) hide
+    (fp_text reference ~ (at 0 -4.5) (layer F.SilkS) hide
       (effects (font (size 1 1) (thickness 0.15)))
     )
-    (fp_text value MountingHole_3.5mm_Pad (at 0 4.5) (layer F.Fab) hide
+    (fp_text value ~ (at 0 4.5) (layer F.Fab) hide
       (effects (font (size 1 1) (thickness 0.15)))
     )
@@
       (effects (font (size 1 1) (thickness 0.15)))
     )
-    (pad 1 thru_hole circle (at 0 0) (size 7 7) (drill 3.5) (layers *.Cu *.Mask))
+    (pad ~ thru_hole circle (at 0 0) (size 7 7) (drill 3.5) (layers *.Cu *.Mask))
   )
   (module MountingHole:MountingHole_3.5mm_Pad (layer F.Cu)
@@
     (tags "mounting hole 3.5mm")
     (attr virtual)
-    (fp_text reference REF** (at 0 -4.5) (layer F.SilkS) hide
+    (fp_text reference ~ (at 0 -4.5) (layer F.SilkS) hide
       (effects (font (size 1 1) (thickness 0.15)))
     )
-    (fp_text value MountingHole_3.5mm_Pad (at 0 4.5) (layer F.Fab) hide
+    (fp_text value ~ (at 0 4.5) (layer F.Fab) hide
       (effects (font (size 1 1) (thickness 0.15)))
     )
@@
     (fp_circle (center 0 0) (end 3.5 0) (layer Cmts.User) (width 0.15))
     (fp_circle (center 0 0) (end 3.75 0) (layer F.CrtYd) (width 0.05))
-    (pad 1 thru_hole circle (at 0 0) (size 7 7) (drill 3.5) (layers *.Cu *.Mask))
+    (pad ~ thru_hole circle (at 0 0) (size 7 7) (drill 3.5) (layers *.Cu *.Mask))
   )
   (module MountingHole:MountingHole_3.5mm_Pad (layer F.Cu)
@@
     (tags "mounting hole 3.5mm")
     (attr virtual)
-    (fp_text reference REF** (at 0 -4.5) (layer F.SilkS) hide
+    (fp_text reference ~ (at 0 -4.5) (layer F.SilkS) hide
       (effects (font (size 1 1) (thickness 0.15)))
     )
-    (fp_text value MountingHole_3.5mm_Pad (at 0 4.5) (layer F.Fab) hide
+    (fp_text value ~ (at 0 4.5) (layer F.Fab) hide
       (effects (font (size 1 1) (thickness 0.15)))
     )
@@
       (effects (font (size 1 1) (thickness 0.15)))
     )
-    (pad 1 thru_hole circle (at 0 0) (size 7 7) (drill 3.5) (layers *.Cu *.Mask))
+    (pad ~ thru_hole circle (at 0 0) (size 7 7) (drill 3.5) (layers *.Cu *.Mask))
   )
   (dimension 123 (width 0.15) (layer Dwgs.User)
