File: template/Hammond_RM2055M/RM2055M.kicad_pcb (KiCad board)
At the start: 2 copper layers, 183 x 128.5 mm, 4 parts

Commit message: feat: Add Templates for Hammond Enclosures
fix mounting hole pad number

Issue #17
Parts:
- ~ (x4): renamed from REF**; value MountingHole_3.5mm_Pad -> ~
Changed lines of the file:
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@@
     (tags "mounting hole 3.5mm")
     (attr virtual)
-    (fp_text reference REF** (at 0 -4.5) (layer F.SilkS) hide
+    (fp_text reference ~ (at 0 -4.5) (layer F.SilkS) hide
       (effects (font (size 1 1) (thickness 0.15)))
     )
-    (fp_text value MountingHole_3.5mm_Pad (at 0 4.5) (layer F.Fab) hide
+    (fp_text value ~ (at 0 4.5) (layer F.Fab) hide
       (effects (font (size 1 1) (thickness 0.15)))
     )
@@
     (tags "mounting hole 3.5mm")
     (attr virtual)
-    (fp_text reference REF** (at 0 -4.5) (layer F.SilkS) hide
+    (fp_text reference ~ (at 0 -4.5) (layer F.SilkS) hide
       (effects (font (size 1 1) (thickness 0.15)))
     )
-    (fp_text value MountingHole_3.5mm_Pad (at 0 4.5) (layer F.Fab) hide
+    (fp_text value ~ (at 0 4.5) (layer F.Fab) hide
       (effects (font (size 1 1) (thickness 0.15)))
     )
@@
     (tags "mounting hole 3.5mm")
     (attr virtual)
-    (fp_text reference REF** (at 0 -4.5) (layer F.SilkS) hide
+    (fp_text reference ~ (at 0 -4.5) (layer F.SilkS) hide
       (effects (font (size 1 1) (thickness 0.15)))
     )
-    (fp_text value MountingHole_3.5mm_Pad (at 0 4.5) (layer F.Fab) hide
+    (fp_text value ~ (at 0 4.5) (layer F.Fab) hide
       (effects (font (size 1 1) (thickness 0.15)))
     )
@@
     (tags "mounting hole 3.5mm")
     (attr virtual)
-    (fp_text reference REF** (at 0 -4.5) (layer F.SilkS) hide
+    (fp_text reference ~ (at 0 -4.5) (layer F.SilkS) hide
       (effects (font (size 1 1) (thickness 0.15)))
     )
-    (fp_text value MountingHole_3.5mm_Pad (at 0 4.5) (layer F.Fab) hide
+    (fp_text value ~ (at 0 4.5) (layer F.Fab) hide
       (effects (font (size 1 1) (thickness 0.15)))
     )
