File: template/Hammond_1598C/1598C.kicad_pcb (KiCad board)
At the start: 2 copper layers, 0 parts

Commit message: feat: Add Templates for Hammond Enclosures
fix origin

Issue #17
Parts:
- added ~: ~, MountingHole:MountingHole_3.5mm_Pad, F.Cu at (26.3, 38.2)
- added ~: ~, MountingHole:MountingHole_3.5mm_Pad, F.Cu at (26.3, 132.4)
- added ~: ~, MountingHole:MountingHole_3.5mm_Pad, F.Cu at (170.6, 38.2)
- added ~: ~, MountingHole:MountingHole_3.5mm_Pad, F.Cu at (170.6, 132.4)
Other:
- board outline added: 166.9 x 140.7 mm
Changed lines of the file:
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@@
   (general
     (thickness 1.6)
-    (drawings 0)
+    (drawings 14)
     (tracks 0)
     (zones 0)
-    (modules 0)
+    (modules 4)
     (nets 1)
   )
@@
     (mod_text_size 1 1)
     (mod_text_width 0.15)
-    (pad_size 1.524 1.524)
-    (pad_drill 0.762)
+    (pad_size 7 7)
+    (pad_drill 3.5)
     (pad_to_mask_clearance 0.051)
     (solder_mask_min_width 0.25)
-    (aux_axis_origin 0 0.5)
+    (aux_axis_origin 0 0)
     (visible_elements 7FFFFFFF)
     (pcbplotparams
@@
     (uvia_drill 0.1)
   )
+  (module MountingHole:MountingHole_3.5mm_Pad (layer F.Cu)
+    (at 26.325 38.25)
+    (descr "Mounting Hole 3.5mm")
+    (tags "mounting hole 3.5mm")
+    (attr virtual)
+    (fp_text reference ~ (at 0 -4.5) (layer F.SilkS) hide
+      (effects (font (size 1 1) (thickness 0.15)))
+    )
+    (fp_text value ~ (at 0 4.5) (layer F.Fab) hide
+      (effects (font (size 1 1) (thickness 0.15)))
+    )
+    (fp_text user %R (at 0.3 0) (layer F.Fab)
+      (effects (font (size 1 1) (thickness 0.15)))
+    )
+    (fp_circle (center 0 0) (end 3.5 0) (layer Cmts.User) (width 0.15))
+    (fp_circle (center 0 0) (end 3.75 0) (layer F.CrtYd) (width 0.05))
+    (pad ~ thru_hole circle (at 0 0) (size 7 7) (drill 3.5) (layers *.Cu *.Mask))
+  )
+  (module MountingHole:MountingHole_3.5mm_Pad (layer F.Cu)
+    (at 26.325 132.45)
+    (descr "Mounting Hole 3.5mm")
+    (tags "mounting hole 3.5mm")
+    (attr virtual)
+    (fp_text reference ~ (at 0 -4.5) (layer F.SilkS) hide
+      (effects (font (size 1 1) (thickness 0.15)))
+    )
+    (fp_text value ~ (at 0 4.5) (layer F.Fab) hide
+      (effects (font (size 1 1) (thickness 0.15)))
+    )
+    (fp_circle (center 0 0) (end 3.75 0) (layer F.CrtYd) (width 0.05))
+    (fp_circle (center 0 0) (end 3.5 0) (layer Cmts.User) (width 0.15))
+    (fp_text user %R (at 0.3 0) (layer F.Fab)
+      (effects (font (size 1 1) (thickness 0.15)))
+    )
+    (pad ~ thru_hole circle (at 0 0) (size 7 7) (drill 3.5) (layers *.Cu *.Mask))
+  )
+  (module MountingHole:MountingHole_3.5mm_Pad (layer F.Cu)
+    (at 170.575 38.25)
+    (descr "Mounting Hole 3.5mm")
+    (tags "mounting hole 3.5mm")
+    (attr virtual)
+    (fp_text reference ~ (at 0 -4.5) (layer F.SilkS) hide
+      (effects (font (size 1 1) (thickness 0.15)))
+    )
+    (fp_text value ~ (at 0 4.5) (layer F.Fab) hide
+      (effects (font (size 1 1) (thickness 0.15)))
+    )
+    (fp_text user %R (at 0.3 0) (layer F.Fab)
+      (effects (font (size 1 1) (thickness 0.15)))
+    )
+    (fp_circle (center 0 0) (end 3.5 0) (layer Cmts.User) (width 0.15))
+    (fp_circle (center 0 0) (end 3.75 0) (layer F.CrtYd) (width 0.05))
+    (pad ~ thru_hole circle (at 0 0) (size 7 7) (drill 3.5) (layers *.Cu *.Mask))
+  )
+  (module MountingHole:MountingHole_3.5mm_Pad (layer F.Cu)
+    (at 170.575 132.45)
+    (descr "Mounting Hole 3.5mm")
+    (tags "mounting hole 3.5mm")
+    (attr virtual)
+    (fp_text reference ~ (at 0 -4.5) (layer F.SilkS) hide
+      (effects (font (size 1 1) (thickness 0.15)))
+    )
+    (fp_text value ~ (at 0 4.5) (layer F.Fab) hide
+      (effects (font (size 1 1) (thickness 0.15)))
+    )
+    (fp_circle (center 0 0) (end 3.75 0) (layer F.CrtYd) (width 0.05))
+    (fp_circle (center 0 0) (end 3.5 0) (layer Cmts.User) (width 0.15))
+    (fp_text user %R (at 0.3 0) (layer F.Fab)
+      (effects (font (size 1 1) (thickness 0.15)))
+    )
+    (pad ~ thru_hole circle (at 0 0) (size 7 7) (drill 3.5) (layers *.Cu *.Mask))
+  )
+  (gr_line (start 104.65 155.7) (end 181.9 155.7) (layer Edge.Cuts) (width 0.05))
+  (gr_arc (start 98.45 151.4) (end 104.65 151.4) (angle -180) (layer Edge.Cuts) (width 0.05))
+  (gr_line (start 92.25 151.4) (end 92.25 155.7) (layer Edge.Cuts) (width 0.05))
+  (gr_line (start 104.65 151.4) (end 104.65 155.7) (layer Edge.Cuts) (width 0.05))
+  (gr_line (start 104.65 15) (end 181.9 15) (layer Edge.Cuts) (width 0.05))
+  (gr_arc (start 98.45 19.3) (end 92.25 19.3) (angle -180) (layer Edge.Cuts) (width 0.05))
+  (gr_line (start 92.25 15) (end 92.25 19.3) (layer Edge.Cuts) (width 0.05))
+  (gr_line (start 104.65 15) (end 104.65 19.3) (layer Edge.Cuts) (width 0.05))
+  (dimension 166.9 (width 0.15) (layer Dwgs.User)
+    (gr_text "166,900 mm" (at 98.45 162) (layer Dwgs.User)
+      (effects (font (size 1 1) (thickness 0.15)))
+    )
+    (feature1 (pts (xy 15 155.7) (xy 15 161.286421)))
+    (feature2 (pts (xy 181.9 155.7) (xy 181.9 161.286421)))
+    (crossbar (pts (xy 181.9 160.7) (xy 15 160.7)))
+    (arrow1a (pts (xy 15 160.7) (xy 16.126504 160.113579)))
+    (arrow1b (pts (xy 15 160.7) (xy 16.126504 161.286421)))
+    (arrow2a (pts (xy 181.9 160.7) (xy 180.773496 160.113579)))
+    (arrow2b (pts (xy 181.9 160.7) (xy 180.773496 161.286421)))
+  )
+  (dimension 140.7 (width 0.15) (layer Dwgs.User)
+    (gr_text "140,700 mm" (at 188.2 85.35 270) (layer Dwgs.User)
+      (effects (font (size 1 1) (thickness 0.15)))
+    )
+    (feature1 (pts (xy 181.9 155.7) (xy 187.486421 155.7)))
+    (feature2 (pts (xy 181.9 15) (xy 187.486421 15)))
+    (crossbar (pts (xy 186.9 15) (xy 186.9 155.7)))
+    (arrow1a (pts (xy 186.9 155.7) (xy 186.313579 154.573496)))
+    (arrow1b (pts (xy 186.9 155.7) (xy 187.486421 154.573496)))
+    (arrow2a (pts (xy 186.9 15) (xy 186.313579 16.126504)))
+    (arrow2b (pts (xy 186.9 15) (xy 187.486421 16.126504)))
+  )
+  (gr_line (start 181.9 155.7) (end 181.9 15) (layer Edge.Cuts) (width 0.05))
+  (gr_line (start 15 15) (end 15 155.7) (layer Edge.Cuts) (width 0.05))
+  (gr_line (start 15 155.7) (end 92.25 155.7) (layer Edge.Cuts) (width 0.05))
+  (gr_line (start 15 15) (end 92.25 15) (layer Edge.Cuts) (width 0.05))
 )
