File: template/Hammond_1598D/1598D.kicad_pcb (KiCad board)
At the start: 2 copper layers, 0 parts

Commit message: feat: Add Templates for Hammond Enclosures
add new board outlines

Issue #17
Parts:
- added ~: ~, MountingHole:MountingHole_3.5mm_Pad, F.Cu at (158.2, 135.8)
- added ~: ~, MountingHole:MountingHole_3.5mm_Pad, F.Cu at (158.2, 85.8)
- added ~: ~, MountingHole:MountingHole_3.5mm_Pad, F.Cu at (158.2, 35.8)
- added ~: ~, MountingHole:MountingHole_3.5mm_Pad, F.Cu at (38.1, 35.8)
- added ~: ~, MountingHole:MountingHole_3.5mm_Pad, F.Cu at (38.1, 185.8)
- added ~: ~, MountingHole:MountingHole_3.5mm_Pad, F.Cu at (38.1, 85.8)
- added ~: ~, MountingHole:MountingHole_3.5mm_Pad, F.Cu at (38.1, 135.8)
- added ~: ~, MountingHole:MountingHole_3.5mm_Pad, F.Cu at (158.2, 185.8)
Other:
- board outline added: 166.3 x 191.5 mm
Changed lines of the file:
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@@
   (general
     (thickness 1.6)
-    (drawings 0)
+    (drawings 14)
     (tracks 0)
     (zones 0)
-    (modules 0)
+    (modules 8)
     (nets 1)
   )
-  (page A4)
+  (page A3)
   (layers
     (0 F.Cu signal)
@@
     (mod_text_size 1 1)
     (mod_text_width 0.15)
-    (pad_size 1.524 1.524)
-    (pad_drill 0.762)
+    (pad_size 7 7)
+    (pad_drill 3.5)
     (pad_to_mask_clearance 0.051)
     (solder_mask_min_width 0.25)
@@
     (uvia_drill 0.1)
   )
+  (module MountingHole:MountingHole_3.5mm_Pad (layer F.Cu)
+    (at 158.225 135.75)
+    (descr "Mounting Hole 3.5mm")
+    (tags "mounting hole 3.5mm")
+    (attr virtual)
+    (fp_text reference ~ (at 0 -4.5) (layer F.SilkS) hide
+      (effects (font (size 1 1) (thickness 0.15)))
+    )
+    (fp_text value ~ (at 0 4.5) (layer F.Fab) hide
+      (effects (font (size 1 1) (thickness 0.15)))
+    )
+    (fp_text user %R (at 0.3 0) (layer F.Fab)
+      (effects (font (size 1 1) (thickness 0.15)))
+    )
+    (fp_circle (center 0 0) (end 3.5 0) (layer Cmts.User) (width 0.15))
+    (fp_circle (center 0 0) (end 3.75 0) (layer F.CrtYd) (width 0.05))
+    (pad ~ thru_hole circle (at 0 0) (size 7 7) (drill 3.5) (layers *.Cu *.Mask))
+  )
+  (module MountingHole:MountingHole_3.5mm_Pad (layer F.Cu)
+    (at 158.225 85.75)
+    (descr "Mounting Hole 3.5mm")
+    (tags "mounting hole 3.5mm")
+    (attr virtual)
+    (fp_text reference ~ (at 0 -4.5) (layer F.SilkS) hide
+      (effects (font (size 1 1) (thickness 0.15)))
+    )
+    (fp_text value ~ (at 0 4.5) (layer F.Fab) hide
+      (effects (font (size 1 1) (thickness 0.15)))
+    )
+    (fp_circle (center 0 0) (end 3.75 0) (layer F.CrtYd) (width 0.05))
+    (fp_circle (center 0 0) (end 3.5 0) (layer Cmts.User) (width 0.15))
+    (fp_text user %R (at 0.3 0) (layer F.Fab)
+      (effects (font (size 1 1) (thickness 0.15)))
+    )
+    (pad ~ thru_hole circle (at 0 0) (size 7 7) (drill 3.5) (layers *.Cu *.Mask))
+  )
+  (module MountingHole:MountingHole_3.5mm_Pad (layer F.Cu)
+    (at 158.225 35.75)
+    (descr "Mounting Hole 3.5mm")
+    (tags "mounting hole 3.5mm")
+    (attr virtual)
+    (fp_text reference ~ (at 0 -4.5) (layer F.SilkS) hide
+      (effects (font (size 1 1) (thickness 0.15)))
+    )
+    (fp_text value ~ (at 0 4.5) (layer F.Fab) hide
+      (effects (font (size 1 1) (thickness 0.15)))
+    )
+    (fp_text user %R (at 0.3 0) (layer F.Fab)
+      (effects (font (size 1 1) (thickness 0.15)))
+    )
+    (fp_circle (center 0 0) (end 3.5 0) (layer Cmts.User) (width 0.15))
+    (fp_circle (center 0 0) (end 3.75 0) (layer F.CrtYd) (width 0.05))
+    (pad ~ thru_hole circle (at 0 0) (size 7 7) (drill 3.5) (layers *.Cu *.Mask))
+  )
+  (module MountingHole:MountingHole_3.5mm_Pad (layer F.Cu)
+    (at 38.075 35.75)
+    (descr "Mounting Hole 3.5mm")
+    (tags "mounting hole 3.5mm")
+    (attr virtual)
+    (fp_text reference ~ (at 0 -4.5) (layer F.SilkS) hide
+      (effects (font (size 1 1) (thickness 0.15)))
+    )
+    (fp_text value ~ (at 0 4.5) (layer F.Fab) hide
+      (effects (font (size 1 1) (thickness 0.15)))
+    )
+    (fp_circle (center 0 0) (end 3.75 0) (layer F.CrtYd) (width 0.05))
+    (fp_circle (center 0 0) (end 3.5 0) (layer Cmts.User) (width 0.15))
+    (fp_text user %R (at 0.3 0) (layer F.Fab)
+      (effects (font (size 1 1) (thickness 0.15)))
+    )
+    (pad ~ thru_hole circle (at 0 0) (size 7 7) (drill 3.5) (layers *.Cu *.Mask))
+  )
+  (module MountingHole:MountingHole_3.5mm_Pad (layer F.Cu)
+    (at 38.075 185.75)
+    (descr "Mounting Hole 3.5mm")
+    (tags "mounting hole 3.5mm")
+    (attr virtual)
+    (fp_text reference ~ (at 0 -4.5) (layer F.SilkS) hide
+      (effects (font (size 1 1) (thickness 0.15)))
+    )
+    (fp_text value ~ (at 0 4.5) (layer F.Fab) hide
+      (effects (font (size 1 1) (thickness 0.15)))
+    )
+    (fp_text user %R (at 0.3 0) (layer F.Fab)
+      (effects (font (size 1 1) (thickness 0.15)))
+    )
+    (fp_circle (center 0 0) (end 3.5 0) (layer Cmts.User) (width 0.15))
+    (fp_circle (center 0 0) (end 3.75 0) (layer F.CrtYd) (width 0.05))
+    (pad ~ thru_hole circle (at 0 0) (size 7 7) (drill 3.5) (layers *.Cu *.Mask))
+  )
+  (module MountingHole:MountingHole_3.5mm_Pad (layer F.Cu)
+    (at 38.075 85.75)
+    (descr "Mounting Hole 3.5mm")
+    (tags "mounting hole 3.5mm")
+    (attr virtual)
+    (fp_text reference ~ (at 0 -4.5) (layer F.SilkS) hide
+      (effects (font (size 1 1) (thickness 0.15)))
+    )
+    (fp_text value ~ (at 0 4.5) (layer F.Fab) hide
+      (effects (font (size 1 1) (thickness 0.15)))
+    )
+    (fp_circle (center 0 0) (end 3.75 0) (layer F.CrtYd) (width 0.05))
+    (fp_circle (center 0 0) (end 3.5 0) (layer Cmts.User) (width 0.15))
+    (fp_text user %R (at 0.3 0) (layer F.Fab)
+      (effects (font (size 1 1) (thickness 0.15)))
+    )
+    (pad ~ thru_hole circle (at 0 0) (size 7 7) (drill 3.5) (layers *.Cu *.Mask))
+  )
+  (module MountingHole:MountingHole_3.5mm_Pad (layer F.Cu)
+    (at 38.075 135.75)
+    (descr "Mounting Hole 3.5mm")
+    (tags "mounting hole 3.5mm")
+    (attr virtual)
+    (fp_text reference ~ (at 0 -4.5) (layer F.SilkS) hide
+      (effects (font (size 1 1) (thickness 0.15)))
+    )
+    (fp_text value ~ (at 0 4.5) (layer F.Fab) hide
+      (effects (font (size 1 1) (thickness 0.15)))
+    )
+    (fp_text user %R (at 0.3 0) (layer F.Fab)
+      (effects (font (size 1 1) (thickness 0.15)))
+    )
+    (fp_circle (center 0 0) (end 3.5 0) (layer Cmts.User) (width 0.15))
+    (fp_circle (center 0 0) (end 3.75 0) (layer F.CrtYd) (width 0.05))
+    (pad ~ thru_hole circle (at 0 0) (size 7 7) (drill 3.5) (layers *.Cu *.Mask))
+  )
+  (module MountingHole:MountingHole_3.5mm_Pad (layer F.Cu)
+    (at 158.225 185.75)
+    (descr "Mounting Hole 3.5mm")
+    (tags "mounting hole 3.5mm")
+    (attr virtual)
+    (fp_text reference ~ (at 0 -4.5) (layer F.SilkS) hide
+      (effects (font (size 1 1) (thickness 0.15)))
+    )
+    (fp_text value ~ (at 0 4.5) (layer F.Fab) hide
+      (effects (font (size 1 1) (thickness 0.15)))
+    )
+    (fp_circle (center 0 0) (end 3.75 0) (layer F.CrtYd) (width 0.05))
+    (fp_circle (center 0 0) (end 3.5 0) (layer Cmts.User) (width 0.15))
+    (fp_text user %R (at 0.3 0) (layer F.Fab)
+      (effects (font (size 1 1) (thickness 0.15)))
+    )
+    (pad ~ thru_hole circle (at 0 0) (size 7 7) (drill 3.5) (layers *.Cu *.Mask))
+  )
+  (gr_arc (start 98.15 202.5) (end 104.15 202.5) (angle -180) (layer Edge.Cuts) (width 0.05))
+  (gr_line (start 104.15 206.5) (end 181.3 206.5) (layer Edge.Cuts) (width 0.05))
+  (gr_line (start 92.15 202.5) (end 92.15 206.5) (layer Edge.Cuts) (width 0.05))
+  (gr_line (start 104.15 202.5) (end 104.15 206.5) (layer Edge.Cuts) (width 0.05))
+  (gr_line (start 104.15 15) (end 181.3 15) (layer Edge.Cuts) (width 0.05))
+  (gr_arc (start 98.15 19) (end 92.15 19) (angle -180) (layer Edge.Cuts) (width 0.05))
+  (gr_line (start 92.15 15) (end 92.15 19) (layer Edge.Cuts) (width 0.05))
+  (gr_line (start 104.15 15) (end 104.15 19) (layer Edge.Cuts) (width 0.05))
+  (dimension 166.3 (width 0.15) (layer Dwgs.User)
+    (gr_text "166,300 mm" (at 98.15 212.8) (layer Dwgs.User)
+      (effects (font (size 1 1) (thickness 0.15)))
+    )
+    (feature1 (pts (xy 15 206.5) (xy 15 212.086421)))
+    (feature2 (pts (xy 181.3 206.5) (xy 181.3 212.086421)))
+    (crossbar (pts (xy 181.3 211.5) (xy 15 211.5)))
+    (arrow1a (pts (xy 15 211.5) (xy 16.126504 210.913579)))
+    (arrow1b (pts (xy 15 211.5) (xy 16.126504 212.086421)))
+    (arrow2a (pts (xy 181.3 211.5) (xy 180.173496 210.913579)))
+    (arrow2b (pts (xy 181.3 211.5) (xy 180.173496 212.086421)))
+  )
+  (dimension 191.5 (width 0.15) (layer Dwgs.User)
+    (gr_text "191,500 mm" (at 187.6 110.75 270) (layer Dwgs.User)
+      (effects (font (size 1 1) (thickness 0.15)))
+    )
+    (feature1 (pts (xy 181.3 206.5) (xy 186.886421 206.5)))
+    (feature2 (pts (xy 181.3 15) (xy 186.886421 15)))
+    (crossbar (pts (xy 186.3 15) (xy 186.3 206.5)))
+    (arrow1a (pts (xy 186.3 206.5) (xy 185.713579 205.373496)))
+    (arrow1b (pts (xy 186.3 206.5) (xy 186.886421 205.373496)))
+    (arrow2a (pts (xy 186.3 15) (xy 185.713579 16.126504)))
+    (arrow2b (pts (xy 186.3 15) (xy 186.886421 16.126504)))
+  )
+  (gr_line (start 181.3 206.5) (end 181.3 15) (layer Edge.Cuts) (width 0.05))
+  (gr_line (start 15 15) (end 15 206.5) (layer Edge.Cuts) (width 0.05))
+  (gr_line (start 15 206.5) (end 92.15 206.5) (layer Edge.Cuts) (width 0.05))
+  (gr_line (start 15 15) (end 92.15 15) (layer Edge.Cuts) (width 0.05))
 )
