File: template/Hammond_1598E/1598E.kicad_pcb (KiCad board)
At the start: 2 copper layers, 0 parts

Commit message: feat: Add Templates for Hammond Enclosures
add new board outlines

Issue #17
Parts:
- added ~: ~, MountingHole:MountingHole_3.5mm_Pad, F.Cu at (133.7, 131.2)
- added ~: ~, MountingHole:MountingHole_3.5mm_Pad, F.Cu at (133.7, 42.4)
- added ~: ~, MountingHole:MountingHole_3.5mm_Pad, F.Cu at (44.8, 131.2)
- added ~: ~, MountingHole:MountingHole_3.5mm_Pad, F.Cu at (44.8, 42.4)
Other:
- board outline added: 148.5 x 143.6 mm
Changed lines of the file:
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@@
   (general
     (thickness 1.6)
-    (drawings 0)
+    (drawings 14)
     (tracks 0)
     (zones 0)
-    (modules 0)
+    (modules 4)
     (nets 1)
   )
@@
     (mod_text_size 1 1)
     (mod_text_width 0.15)
-    (pad_size 1.524 1.524)
-    (pad_drill 0.762)
+    (pad_size 7 7)
+    (pad_drill 3.5)
     (pad_to_mask_clearance 0.051)
     (solder_mask_min_width 0.25)
@@
     (uvia_drill 0.1)
   )
+  (module MountingHole:MountingHole_3.5mm_Pad (layer F.Cu)
+    (at 133.725 131.215)
+    (descr "Mounting Hole 3.5mm")
+    (tags "mounting hole 3.5mm")
+    (attr virtual)
+    (fp_text reference ~ (at 0 -4.5) (layer F.SilkS) hide
+      (effects (font (size 1 1) (thickness 0.15)))
+    )
+    (fp_text value ~ (at 0 4.5) (layer F.Fab) hide
+      (effects (font (size 1 1) (thickness 0.15)))
+    )
+    (fp_text user %R (at 0.3 0) (layer F.Fab)
+      (effects (font (size 1 1) (thickness 0.15)))
+    )
+    (fp_circle (center 0 0) (end 3.5 0) (layer Cmts.User) (width 0.15))
+    (fp_circle (center 0 0) (end 3.75 0) (layer F.CrtYd) (width 0.05))
+    (pad ~ thru_hole circle (at 0 0) (size 7 7) (drill 3.5) (layers *.Cu *.Mask))
+  )
+  (module MountingHole:MountingHole_3.5mm_Pad (layer F.Cu)
+    (at 133.725 42.385)
+    (descr "Mounting Hole 3.5mm")
+    (tags "mounting hole 3.5mm")
+    (attr virtual)
+    (fp_text reference ~ (at 0 -4.5) (layer F.SilkS) hide
+      (effects (font (size 1 1) (thickness 0.15)))
+    )
+    (fp_text value ~ (at 0 4.5) (layer F.Fab) hide
+      (effects (font (size 1 1) (thickness 0.15)))
+    )
+    (fp_circle (center 0 0) (end 3.75 0) (layer F.CrtYd) (width 0.05))
+    (fp_circle (center 0 0) (end 3.5 0) (layer Cmts.User) (width 0.15))
+    (fp_text user %R (at 0.3 0) (layer F.Fab)
+      (effects (font (size 1 1) (thickness 0.15)))
+    )
+    (pad ~ thru_hole circle (at 0 0) (size 7 7) (drill 3.5) (layers *.Cu *.Mask))
+  )
+  (module MountingHole:MountingHole_3.5mm_Pad (layer F.Cu)
+    (at 44.775 131.215)
+    (descr "Mounting Hole 3.5mm")
+    (tags "mounting hole 3.5mm")
+    (attr virtual)
+    (fp_text reference ~ (at 0 -4.5) (layer F.SilkS) hide
+      (effects (font (size 1 1) (thickness 0.15)))
+    )
+    (fp_text value ~ (at 0 4.5) (layer F.Fab) hide
+      (effects (font (size 1 1) (thickness 0.15)))
+    )
+    (fp_text user %R (at 0.3 0) (layer F.Fab)
+      (effects (font (size 1 1) (thickness 0.15)))
+    )
+    (fp_circle (center 0 0) (end 3.5 0) (layer Cmts.User) (width 0.15))
+    (fp_circle (center 0 0) (end 3.75 0) (layer F.CrtYd) (width 0.05))
+    (pad ~ thru_hole circle (at 0 0) (size 7 7) (drill 3.5) (layers *.Cu *.Mask))
+  )
+  (module MountingHole:MountingHole_3.5mm_Pad (layer F.Cu)
+    (at 44.775 42.385)
+    (descr "Mounting Hole 3.5mm")
+    (tags "mounting hole 3.5mm")
+    (attr virtual)
+    (fp_text reference ~ (at 0 -4.5) (layer F.SilkS) hide
+      (effects (font (size 1 1) (thickness 0.15)))
+    )
+    (fp_text value ~ (at 0 4.5) (layer F.Fab) hide
+      (effects (font (size 1 1) (thickness 0.15)))
+    )
+    (fp_circle (center 0 0) (end 3.75 0) (layer F.CrtYd) (width 0.05))
+    (fp_circle (center 0 0) (end 3.5 0) (layer Cmts.User) (width 0.15))
+    (fp_text user %R (at 0.3 0) (layer F.Fab)
+      (effects (font (size 1 1) (thickness 0.15)))
+    )
+    (pad ~ thru_hole circle (at 0 0) (size 7 7) (drill 3.5) (layers *.Cu *.Mask))
+  )
+  (gr_arc (start 89.25 154.9) (end 95.55 154.9) (angle -180) (layer Edge.Cuts) (width 0.05))
+  (gr_line (start 95.55 158.6) (end 163.5 158.6) (layer Edge.Cuts) (width 0.05))
+  (gr_line (start 82.95 154.9) (end 82.95 158.6) (layer Edge.Cuts) (width 0.05))
+  (gr_line (start 95.55 154.9) (end 95.55 158.6) (layer Edge.Cuts) (width 0.05))
+  (gr_arc (start 89.25 18.7) (end 82.95 18.7) (angle -180) (layer Edge.Cuts) (width 0.05))
+  (gr_line (start 95.55 15) (end 163.5 15) (layer Edge.Cuts) (width 0.05))
+  (gr_line (start 82.95 15) (end 82.95 18.7) (layer Edge.Cuts) (width 0.05))
+  (gr_line (start 95.55 15) (end 95.55 18.7) (layer Edge.Cuts) (width 0.05))
+  (dimension 148.5 (width 0.15) (layer Dwgs.User)
+    (gr_text "148,500 mm" (at 89.25 164.3) (layer Dwgs.User)
+      (effects (font (size 1 1) (thickness 0.15)))
+    )
+    (feature1 (pts (xy 15 158.6) (xy 15 163.586421)))
+    (feature2 (pts (xy 163.5 158.6) (xy 163.5 163.586421)))
+    (crossbar (pts (xy 163.5 163) (xy 15 163)))
+    (arrow1a (pts (xy 15 163) (xy 16.126504 162.413579)))
+    (arrow1b (pts (xy 15 163) (xy 16.126504 163.586421)))
+    (arrow2a (pts (xy 163.5 163) (xy 162.373496 162.413579)))
+    (arrow2b (pts (xy 163.5 163) (xy 162.373496 163.586421)))
+  )
+  (dimension 143.6 (width 0.15) (layer Dwgs.User)
+    (gr_text "143,600 mm" (at 169.8 86.8 270) (layer Dwgs.User)
+      (effects (font (size 1 1) (thickness 0.15)))
+    )
+    (feature1 (pts (xy 163.5 158.6) (xy 169.086421 158.6)))
+    (feature2 (pts (xy 163.5 15) (xy 169.086421 15)))
+    (crossbar (pts (xy 168.5 15) (xy 168.5 158.6)))
+    (arrow1a (pts (xy 168.5 158.6) (xy 167.913579 157.473496)))
+    (arrow1b (pts (xy 168.5 158.6) (xy 169.086421 157.473496)))
+    (arrow2a (pts (xy 168.5 15) (xy 167.913579 16.126504)))
+    (arrow2b (pts (xy 168.5 15) (xy 169.086421 16.126504)))
+  )
+  (gr_line (start 163.5 158.6) (end 163.5 15) (layer Edge.Cuts) (width 0.05))
+  (gr_line (start 15 15) (end 15 158.6) (layer Edge.Cuts) (width 0.05))
+  (gr_line (start 15 158.6) (end 82.95 158.6) (layer Edge.Cuts) (width 0.05))
+  (gr_line (start 15 15) (end 82.95 15) (layer Edge.Cuts) (width 0.05))
 )
