File: template/Hammond_1598F/1598F.kicad_pcb (KiCad board)
At the start: 2 copper layers, 0 parts

Commit message: feat: Add Templates for Hammond Enclosures
add new board outlines

Issue #17
Parts:
- added ~: ~, MountingHole:MountingHole_3.5mm_Pad, F.Cu at (57.5, 43.1)
- added ~: ~, MountingHole:MountingHole_3.5mm_Pad, F.Cu at (57.5, 131.6)
- added ~: ~, MountingHole:MountingHole_3.5mm_Pad, F.Cu at (210.9, 43.1)
- added ~: ~, MountingHole:MountingHole_3.5mm_Pad, F.Cu at (210.9, 131.6)
Other:
- board outline added: 238.3 x 144.8 mm
Changed lines of the file:
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@@
   (general
     (thickness 1.6)
-    (drawings 0)
+    (drawings 14)
     (tracks 0)
     (zones 0)
-    (modules 0)
+    (modules 4)
     (nets 1)
   )
@@
     (mod_text_size 1 1)
     (mod_text_width 0.15)
-    (pad_size 1.524 1.524)
-    (pad_drill 0.762)
+    (pad_size 7 7)
+    (pad_drill 3.5)
     (pad_to_mask_clearance 0.051)
     (solder_mask_min_width 0.25)
@@
     (uvia_drill 0.1)
   )
+  (module MountingHole:MountingHole_3.5mm_Pad (layer F.Cu)
+    (at 57.475 43.1)
+    (descr "Mounting Hole 3.5mm")
+    (tags "mounting hole 3.5mm")
+    (attr virtual)
+    (fp_text reference ~ (at 0 -4.5) (layer F.SilkS) hide
+      (effects (font (size 1 1) (thickness 0.15)))
+    )
+    (fp_text value ~ (at 0 4.5) (layer F.Fab) hide
+      (effects (font (size 1 1) (thickness 0.15)))
+    )
+    (fp_text user %R (at 0.3 0) (layer F.Fab)
+      (effects (font (size 1 1) (thickness 0.15)))
+    )
+    (fp_circle (center 0 0) (end 3.5 0) (layer Cmts.User) (width 0.15))
+    (fp_circle (center 0 0) (end 3.75 0) (layer F.CrtYd) (width 0.05))
+    (pad ~ thru_hole circle (at 0 0) (size 7 7) (drill 3.5) (layers *.Cu *.Mask))
+  )
+  (module MountingHole:MountingHole_3.5mm_Pad (layer F.Cu)
+    (at 57.475 131.6)
+    (descr "Mounting Hole 3.5mm")
+    (tags "mounting hole 3.5mm")
+    (attr virtual)
+    (fp_text reference ~ (at 0 -4.5) (layer F.SilkS) hide
+      (effects (font (size 1 1) (thickness 0.15)))
+    )
+    (fp_text value ~ (at 0 4.5) (layer F.Fab) hide
+      (effects (font (size 1 1) (thickness 0.15)))
+    )
+    (fp_circle (center 0 0) (end 3.75 0) (layer F.CrtYd) (width 0.05))
+    (fp_circle (center 0 0) (end 3.5 0) (layer Cmts.User) (width 0.15))
+    (fp_text user %R (at 0.3 0) (layer F.Fab)
+      (effects (font (size 1 1) (thickness 0.15)))
+    )
+    (pad ~ thru_hole circle (at 0 0) (size 7 7) (drill 3.5) (layers *.Cu *.Mask))
+  )
+  (module MountingHole:MountingHole_3.5mm_Pad (layer F.Cu)
+    (at 210.875 43.1)
+    (descr "Mounting Hole 3.5mm")
+    (tags "mounting hole 3.5mm")
+    (attr virtual)
+    (fp_text reference ~ (at 0 -4.5) (layer F.SilkS) hide
+      (effects (font (size 1 1) (thickness 0.15)))
+    )
+    (fp_text value ~ (at 0 4.5) (layer F.Fab) hide
+      (effects (font (size 1 1) (thickness 0.15)))
+    )
+    (fp_text user %R (at 0.3 0) (layer F.Fab)
+      (effects (font (size 1 1) (thickness 0.15)))
+    )
+    (fp_circle (center 0 0) (end 3.5 0) (layer Cmts.User) (width 0.15))
+    (fp_circle (center 0 0) (end 3.75 0) (layer F.CrtYd) (width 0.05))
+    (pad ~ thru_hole circle (at 0 0) (size 7 7) (drill 3.5) (layers *.Cu *.Mask))
+  )
+  (module MountingHole:MountingHole_3.5mm_Pad (layer F.Cu)
+    (at 210.875 131.6)
+    (descr "Mounting Hole 3.5mm")
+    (tags "mounting hole 3.5mm")
+    (attr virtual)
+    (fp_text reference ~ (at 0 -4.5) (layer F.SilkS) hide
+      (effects (font (size 1 1) (thickness 0.15)))
+    )
+    (fp_text value ~ (at 0 4.5) (layer F.Fab) hide
+      (effects (font (size 1 1) (thickness 0.15)))
+    )
+    (fp_circle (center 0 0) (end 3.75 0) (layer F.CrtYd) (width 0.05))
+    (fp_circle (center 0 0) (end 3.5 0) (layer Cmts.User) (width 0.15))
+    (fp_text user %R (at 0.3 0) (layer F.Fab)
+      (effects (font (size 1 1) (thickness 0.15)))
+    )
+    (pad ~ thru_hole circle (at 0 0) (size 7 7) (drill 3.5) (layers *.Cu *.Mask))
+  )
+  (gr_arc (start 134.175 156.8) (end 140.175 156.8) (angle -180) (layer Edge.Cuts) (width 0.05))
+  (gr_line (start 140.175 159.8) (end 253.35 159.8) (layer Edge.Cuts) (width 0.05))
+  (gr_line (start 128.175 156.8) (end 128.175 159.8) (layer Edge.Cuts) (width 0.05))
+  (gr_line (start 140.175 156.8) (end 140.175 159.8) (layer Edge.Cuts) (width 0.05))
+  (gr_arc (start 134.175 18) (end 128.175 18) (angle -180) (layer Edge.Cuts) (width 0.05))
+  (gr_line (start 140.175 15) (end 253.35 15) (layer Edge.Cuts) (width 0.05))
+  (gr_line (start 128.175 15) (end 128.175 18) (layer Edge.Cuts) (width 0.05))
+  (gr_line (start 140.175 15) (end 140.175 18) (layer Edge.Cuts) (width 0.05))
+  (dimension 238.35 (width 0.15) (layer Dwgs.User)
+    (gr_text "238,350 mm" (at 134.175 166.3) (layer Dwgs.User)
+      (effects (font (size 1 1) (thickness 0.15)))
+    )
+    (feature1 (pts (xy 15 159.8) (xy 15 165.586421)))
+    (feature2 (pts (xy 253.35 159.8) (xy 253.35 165.586421)))
+    (crossbar (pts (xy 253.35 165) (xy 15 165)))
+    (arrow1a (pts (xy 15 165) (xy 16.126504 164.413579)))
+    (arrow1b (pts (xy 15 165) (xy 16.126504 165.586421)))
+    (arrow2a (pts (xy 253.35 165) (xy 252.223496 164.413579)))
+    (arrow2b (pts (xy 253.35 165) (xy 252.223496 165.586421)))
+  )
+  (dimension 144.8 (width 0.15) (layer Dwgs.User)
+    (gr_text "144,800 mm" (at 259.8 87.4 270) (layer Dwgs.User)
+      (effects (font (size 1 1) (thickness 0.15)))
+    )
+    (feature1 (pts (xy 253.35 159.8) (xy 259.086421 159.8)))
+    (feature2 (pts (xy 253.35 15) (xy 259.086421 15)))
+    (crossbar (pts (xy 258.5 15) (xy 258.5 159.8)))
+    (arrow1a (pts (xy 258.5 159.8) (xy 257.913579 158.673496)))
+    (arrow1b (pts (xy 258.5 159.8) (xy 259.086421 158.673496)))
+    (arrow2a (pts (xy 258.5 15) (xy 257.913579 16.126504)))
+    (arrow2b (pts (xy 258.5 15) (xy 259.086421 16.126504)))
+  )
+  (gr_line (start 253.35 159.8) (end 253.35 15) (layer Edge.Cuts) (width 0.05))
+  (gr_line (start 15 15) (end 15 159.8) (layer Edge.Cuts) (width 0.05))
+  (gr_line (start 15 159.8) (end 128.175 159.8) (layer Edge.Cuts) (width 0.05))
+  (gr_line (start 15 15) (end 128.175 15) (layer Edge.Cuts) (width 0.05))
 )
