File: template/Hammond_1598G/1598G.kicad_pcb (KiCad board)
At the start: 2 copper layers, 0 parts

Commit message: feat: Add Templates for Hammond Enclosures
add new board outlines

Issue #17
Parts:
- added ~: ~, MountingHole:MountingHole_3.5mm_Pad, F.Cu at (57.4, 42.4)
- added ~: ~, MountingHole:MountingHole_3.5mm_Pad, F.Cu at (57.4, 131.2)
- added ~: ~, MountingHole:MountingHole_3.5mm_Pad, F.Cu at (211.1, 42.4)
- added ~: ~, MountingHole:MountingHole_3.5mm_Pad, F.Cu at (211.1, 131.2)
Other:
- board outline added: 238.5 x 143.6 mm
Changed lines of the file:
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@@
   (general
     (thickness 1.6)
-    (drawings 0)
+    (drawings 14)
     (tracks 0)
     (zones 0)
-    (modules 0)
+    (modules 4)
     (nets 1)
   )
@@
     (mod_text_size 1 1)
     (mod_text_width 0.15)
-    (pad_size 1.524 1.524)
-    (pad_drill 0.762)
+    (pad_size 7 7)
+    (pad_drill 3.5)
     (pad_to_mask_clearance 0.051)
     (solder_mask_min_width 0.25)
@@
     (uvia_drill 0.1)
   )
+  (module MountingHole:MountingHole_3.5mm_Pad (layer F.Cu)
+    (at 57.4 42.35)
+    (descr "Mounting Hole 3.5mm")
+    (tags "mounting hole 3.5mm")
+    (attr virtual)
+    (fp_text reference ~ (at 0 -4.5) (layer F.SilkS) hide
+      (effects (font (size 1 1) (thickness 0.15)))
+    )
+    (fp_text value ~ (at 0 4.5) (layer F.Fab) hide
+      (effects (font (size 1 1) (thickness 0.15)))
+    )
+    (fp_text user %R (at 0.3 0) (layer F.Fab)
+      (effects (font (size 1 1) (thickness 0.15)))
+    )
+    (fp_circle (center 0 0) (end 3.5 0) (layer Cmts.User) (width 0.15))
+    (fp_circle (center 0 0) (end 3.75 0) (layer F.CrtYd) (width 0.05))
+    (pad ~ thru_hole circle (at 0 0) (size 7 7) (drill 3.5) (layers *.Cu *.Mask))
+  )
+  (module MountingHole:MountingHole_3.5mm_Pad (layer F.Cu)
+    (at 57.4 131.25)
+    (descr "Mounting Hole 3.5mm")
+    (tags "mounting hole 3.5mm")
+    (attr virtual)
+    (fp_text reference ~ (at 0 -4.5) (layer F.SilkS) hide
+      (effects (font (size 1 1) (thickness 0.15)))
+    )
+    (fp_text value ~ (at 0 4.5) (layer F.Fab) hide
+      (effects (font (size 1 1) (thickness 0.15)))
+    )
+    (fp_circle (center 0 0) (end 3.75 0) (layer F.CrtYd) (width 0.05))
+    (fp_circle (center 0 0) (end 3.5 0) (layer Cmts.User) (width 0.15))
+    (fp_text user %R (at 0.3 0) (layer F.Fab)
+      (effects (font (size 1 1) (thickness 0.15)))
+    )
+    (pad ~ thru_hole circle (at 0 0) (size 7 7) (drill 3.5) (layers *.Cu *.Mask))
+  )
+  (module MountingHole:MountingHole_3.5mm_Pad (layer F.Cu)
+    (at 211.1 42.35)
+    (descr "Mounting Hole 3.5mm")
+    (tags "mounting hole 3.5mm")
+    (attr virtual)
+    (fp_text reference ~ (at 0 -4.5) (layer F.SilkS) hide
+      (effects (font (size 1 1) (thickness 0.15)))
+    )
+    (fp_text value ~ (at 0 4.5) (layer F.Fab) hide
+      (effects (font (size 1 1) (thickness 0.15)))
+    )
+    (fp_text user %R (at 0.3 0) (layer F.Fab)
+      (effects (font (size 1 1) (thickness 0.15)))
+    )
+    (fp_circle (center 0 0) (end 3.5 0) (layer Cmts.User) (width 0.15))
+    (fp_circle (center 0 0) (end 3.75 0) (layer F.CrtYd) (width 0.05))
+    (pad ~ thru_hole circle (at 0 0) (size 7 7) (drill 3.5) (layers *.Cu *.Mask))
+  )
+  (module MountingHole:MountingHole_3.5mm_Pad (layer F.Cu)
+    (at 211.1 131.25)
+    (descr "Mounting Hole 3.5mm")
+    (tags "mounting hole 3.5mm")
+    (attr virtual)
+    (fp_text reference ~ (at 0 -4.5) (layer F.SilkS) hide
+      (effects (font (size 1 1) (thickness 0.15)))
+    )
+    (fp_text value ~ (at 0 4.5) (layer F.Fab) hide
+      (effects (font (size 1 1) (thickness 0.15)))
+    )
+    (fp_circle (center 0 0) (end 3.75 0) (layer F.CrtYd) (width 0.05))
+    (fp_circle (center 0 0) (end 3.5 0) (layer Cmts.User) (width 0.15))
+    (fp_text user %R (at 0.3 0) (layer F.Fab)
+      (effects (font (size 1 1) (thickness 0.15)))
+    )
+    (pad ~ thru_hole circle (at 0 0) (size 7 7) (drill 3.5) (layers *.Cu *.Mask))
+  )
+  (gr_arc (start 134.25 155.9) (end 140.55 155.9) (angle -180) (layer Edge.Cuts) (width 0.05))
+  (gr_line (start 140.55 158.6) (end 253.5 158.6) (layer Edge.Cuts) (width 0.05))
+  (gr_line (start 127.95 155.9) (end 127.95 158.6) (layer Edge.Cuts) (width 0.05))
+  (gr_line (start 140.55 155.9) (end 140.55 158.6) (layer Edge.Cuts) (width 0.05))
+  (gr_arc (start 134.25 17.7) (end 127.95 17.7) (angle -180) (layer Edge.Cuts) (width 0.05))
+  (gr_line (start 140.55 15) (end 253.5 15) (layer Edge.Cuts) (width 0.05))
+  (gr_line (start 127.95 15) (end 127.95 17.7) (layer Edge.Cuts) (width 0.05))
+  (gr_line (start 140.55 15) (end 140.55 17.7) (layer Edge.Cuts) (width 0.05))
+  (dimension 238.5 (width 0.15) (layer Dwgs.User)
+    (gr_text "238,500 mm" (at 134.25 164.8) (layer Dwgs.User)
+      (effects (font (size 1 1) (thickness 0.15)))
+    )
+    (feature1 (pts (xy 15 158.6) (xy 15 164.086421)))
+    (feature2 (pts (xy 253.5 158.6) (xy 253.5 164.086421)))
+    (crossbar (pts (xy 253.5 163.5) (xy 15 163.5)))
+    (arrow1a (pts (xy 15 163.5) (xy 16.126504 162.913579)))
+    (arrow1b (pts (xy 15 163.5) (xy 16.126504 164.086421)))
+    (arrow2a (pts (xy 253.5 163.5) (xy 252.373496 162.913579)))
+    (arrow2b (pts (xy 253.5 163.5) (xy 252.373496 164.086421)))
+  )
+  (dimension 143.6 (width 0.15) (layer Dwgs.User)
+    (gr_text "143,600 mm" (at 259.8 86.8 270) (layer Dwgs.User)
+      (effects (font (size 1 1) (thickness 0.15)))
+    )
+    (feature1 (pts (xy 253.5 158.6) (xy 259.086421 158.6)))
+    (feature2 (pts (xy 253.5 15) (xy 259.086421 15)))
+    (crossbar (pts (xy 258.5 15) (xy 258.5 158.6)))
+    (arrow1a (pts (xy 258.5 158.6) (xy 257.913579 157.473496)))
+    (arrow1b (pts (xy 258.5 158.6) (xy 259.086421 157.473496)))
+    (arrow2a (pts (xy 258.5 15) (xy 257.913579 16.126504)))
+    (arrow2b (pts (xy 258.5 15) (xy 259.086421 16.126504)))
+  )
+  (gr_line (start 253.5 158.6) (end 253.5 15) (layer Edge.Cuts) (width 0.05))
+  (gr_line (start 15 15) (end 15 158.6) (layer Edge.Cuts) (width 0.05))
+  (gr_line (start 15 158.6) (end 127.95 158.6) (layer Edge.Cuts) (width 0.05))
+  (gr_line (start 15 15) (end 127.95 15) (layer Edge.Cuts) (width 0.05))
 )
