File: template/Hammond_1598H/1598H.kicad_pcb (KiCad board)
At the start: 2 copper layers, 0 parts

Commit message: feat: Add Templates for Hammond Enclosures
add new board outlines

Issue #17
Parts:
- added ~: ~, MountingHole:MountingHole_3.5mm_Pad, F.Cu at (260.6, 30.1)
- added ~: ~, MountingHole:MountingHole_3.5mm_Pad, F.Cu at (260.6, 184.2)
- added ~: ~, MountingHole:MountingHole_3.5mm_Pad, F.Cu at (38.1, 184.2)
- added ~: ~, MountingHole:MountingHole_3.5mm_Pad, F.Cu at (38.1, 30.1)
- added ~: ~, MountingHole:MountingHole_3.5mm_Pad, F.Cu at (127.1, 184.2)
- added ~: ~, MountingHole:MountingHole_3.5mm_Pad, F.Cu at (127.1, 30.1)
- added ~: ~, MountingHole:MountingHole_3.5mm_Pad, F.Cu at (171.6, 184.2)
- added ~: ~, MountingHole:MountingHole_3.5mm_Pad, F.Cu at (171.6, 30.1)
Other:
- board outline added: 268.7 x 184.3 mm
Changed lines of the file:
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@@
   (general
     (thickness 1.6)
-    (drawings 0)
+    (drawings 14)
     (tracks 0)
     (zones 0)
-    (modules 0)
+    (modules 8)
     (nets 1)
   )
-  (page A4)
+  (page A3)
   (layers
     (0 F.Cu signal)
@@
     (mod_text_size 1 1)
     (mod_text_width 0.15)
-    (pad_size 1.524 1.524)
-    (pad_drill 0.762)
+    (pad_size 7 7)
+    (pad_drill 3.5)
     (pad_to_mask_clearance 0.051)
     (solder_mask_min_width 0.25)
@@
     (uvia_drill 0.1)
   )
+  (module MountingHole:MountingHole_3.5mm_Pad (layer F.Cu)
+    (at 260.6 30.15)
+    (descr "Mounting Hole 3.5mm")
+    (tags "mounting hole 3.5mm")
+    (attr virtual)
+    (fp_text reference ~ (at 0 -4.5) (layer F.SilkS) hide
+      (effects (font (size 1 1) (thickness 0.15)))
+    )
+    (fp_text value ~ (at 0 4.5) (layer F.Fab) hide
+      (effects (font (size 1 1) (thickness 0.15)))
+    )
+    (fp_text user %R (at 0.3 0) (layer F.Fab)
+      (effects (font (size 1 1) (thickness 0.15)))
+    )
+    (fp_circle (center 0 0) (end 3.5 0) (layer Cmts.User) (width 0.15))
+    (fp_circle (center 0 0) (end 3.75 0) (layer F.CrtYd) (width 0.05))
+    (pad ~ thru_hole circle (at 0 0) (size 7 7) (drill 3.5) (layers *.Cu *.Mask))
+  )
+  (module MountingHole:MountingHole_3.5mm_Pad (layer F.Cu)
+    (at 260.6 184.15)
+    (descr "Mounting Hole 3.5mm")
+    (tags "mounting hole 3.5mm")
+    (attr virtual)
+    (fp_text reference ~ (at 0 -4.5) (layer F.SilkS) hide
+      (effects (font (size 1 1) (thickness 0.15)))
+    )
+    (fp_text value ~ (at 0 4.5) (layer F.Fab) hide
+      (effects (font (size 1 1) (thickness 0.15)))
+    )
+    (fp_circle (center 0 0) (end 3.75 0) (layer F.CrtYd) (width 0.05))
+    (fp_circle (center 0 0) (end 3.5 0) (layer Cmts.User) (width 0.15))
+    (fp_text user %R (at 0.3 0) (layer F.Fab)
+      (effects (font (size 1 1) (thickness 0.15)))
+    )
+    (pad ~ thru_hole circle (at 0 0) (size 7 7) (drill 3.5) (layers *.Cu *.Mask))
+  )
+  (module MountingHole:MountingHole_3.5mm_Pad (layer F.Cu)
+    (at 38.1 184.15)
+    (descr "Mounting Hole 3.5mm")
+    (tags "mounting hole 3.5mm")
+    (attr virtual)
+    (fp_text reference ~ (at 0 -4.5) (layer F.SilkS) hide
+      (effects (font (size 1 1) (thickness 0.15)))
+    )
+    (fp_text value ~ (at 0 4.5) (layer F.Fab) hide
+      (effects (font (size 1 1) (thickness 0.15)))
+    )
+    (fp_circle (center 0 0) (end 3.75 0) (layer F.CrtYd) (width 0.05))
+    (fp_circle (center 0 0) (end 3.5 0) (layer Cmts.User) (width 0.15))
+    (fp_text user %R (at 0.3 0) (layer F.Fab)
+      (effects (font (size 1 1) (thickness 0.15)))
+    )
+    (pad ~ thru_hole circle (at 0 0) (size 7 7) (drill 3.5) (layers *.Cu *.Mask))
+  )
+  (module MountingHole:MountingHole_3.5mm_Pad (layer F.Cu)
+    (at 38.1 30.15)
+    (descr "Mounting Hole 3.5mm")
+    (tags "mounting hole 3.5mm")
+    (attr virtual)
+    (fp_text reference ~ (at 0 -4.5) (layer F.SilkS) hide
+      (effects (font (size 1 1) (thickness 0.15)))
+    )
+    (fp_text value ~ (at 0 4.5) (layer F.Fab) hide
+      (effects (font (size 1 1) (thickness 0.15)))
+    )
+    (fp_text user %R (at 0.3 0) (layer F.Fab)
+      (effects (font (size 1 1) (thickness 0.15)))
+    )
+    (fp_circle (center 0 0) (end 3.5 0) (layer Cmts.User) (width 0.15))
+    (fp_circle (center 0 0) (end 3.75 0) (layer F.CrtYd) (width 0.05))
+    (pad ~ thru_hole circle (at 0 0) (size 7 7) (drill 3.5) (layers *.Cu *.Mask))
+  )
+  (module MountingHole:MountingHole_3.5mm_Pad (layer F.Cu)
+    (at 127.1 184.15)
+    (descr "Mounting Hole 3.5mm")
+    (tags "mounting hole 3.5mm")
+    (attr virtual)
+    (fp_text reference ~ (at 0 -4.5) (layer F.SilkS) hide
+      (effects (font (size 1 1) (thickness 0.15)))
+    )
+    (fp_text value ~ (at 0 4.5) (layer F.Fab) hide
+      (effects (font (size 1 1) (thickness 0.15)))
+    )
+    (fp_text user %R (at 0.3 0) (layer F.Fab)
+      (effects (font (size 1 1) (thickness 0.15)))
+    )
+    (fp_circle (center 0 0) (end 3.5 0) (layer Cmts.User) (width 0.15))
+    (fp_circle (center 0 0) (end 3.75 0) (layer F.CrtYd) (width 0.05))
+    (pad ~ thru_hole circle (at 0 0) (size 7 7) (drill 3.5) (layers *.Cu *.Mask))
+  )
+  (module MountingHole:MountingHole_3.5mm_Pad (layer F.Cu)
+    (at 127.1 30.15)
+    (descr "Mounting Hole 3.5mm")
+    (tags "mounting hole 3.5mm")
+    (attr virtual)
+    (fp_text reference ~ (at 0 -4.5) (layer F.SilkS) hide
+      (effects (font (size 1 1) (thickness 0.15)))
+    )
+    (fp_text value ~ (at 0 4.5) (layer F.Fab) hide
+      (effects (font (size 1 1) (thickness 0.15)))
+    )
+    (fp_circle (center 0 0) (end 3.75 0) (layer F.CrtYd) (width 0.05))
+    (fp_circle (center 0 0) (end 3.5 0) (layer Cmts.User) (width 0.15))
+    (fp_text user %R (at 0.3 0) (layer F.Fab)
+      (effects (font (size 1 1) (thickness 0.15)))
+    )
+    (pad ~ thru_hole circle (at 0 0) (size 7 7) (drill 3.5) (layers *.Cu *.Mask))
+  )
+  (module MountingHole:MountingHole_3.5mm_Pad (layer F.Cu)
+    (at 171.6 184.15)
+    (descr "Mounting Hole 3.5mm")
+    (tags "mounting hole 3.5mm")
+    (attr virtual)
+    (fp_text reference ~ (at 0 -4.5) (layer F.SilkS) hide
+      (effects (font (size 1 1) (thickness 0.15)))
+    )
+    (fp_text value ~ (at 0 4.5) (layer F.Fab) hide
+      (effects (font (size 1 1) (thickness 0.15)))
+    )
+    (fp_text user %R (at 0.3 0) (layer F.Fab)
+      (effects (font (size 1 1) (thickness 0.15)))
+    )
+    (fp_circle (center 0 0) (end 3.5 0) (layer Cmts.User) (width 0.15))
+    (fp_circle (center 0 0) (end 3.75 0) (layer F.CrtYd) (width 0.05))
+    (pad ~ thru_hole circle (at 0 0) (size 7 7) (drill 3.5) (layers *.Cu *.Mask))
+  )
+  (module MountingHole:MountingHole_3.5mm_Pad (layer F.Cu)
+    (at 171.6 30.15)
+    (descr "Mounting Hole 3.5mm")
+    (tags "mounting hole 3.5mm")
+    (attr virtual)
+    (fp_text reference ~ (at 0 -4.5) (layer F.SilkS) hide
+      (effects (font (size 1 1) (thickness 0.15)))
+    )
+    (fp_text value ~ (at 0 4.5) (layer F.Fab) hide
+      (effects (font (size 1 1) (thickness 0.15)))
+    )
+    (fp_circle (center 0 0) (end 3.75 0) (layer F.CrtYd) (width 0.05))
+    (fp_circle (center 0 0) (end 3.5 0) (layer Cmts.User) (width 0.15))
+    (fp_text user %R (at 0.3 0) (layer F.Fab)
+      (effects (font (size 1 1) (thickness 0.15)))
+    )
+    (pad ~ thru_hole circle (at 0 0) (size 7 7) (drill 3.5) (layers *.Cu *.Mask))
+  )
+  (gr_arc (start 149.35 196.5) (end 155.55 196.5) (angle -180) (layer Edge.Cuts) (width 0.05))
+  (gr_line (start 155.55 199.3) (end 283.7 199.3) (layer Edge.Cuts) (width 0.05))
+  (gr_line (start 143.15 196.5) (end 143.15 199.3) (layer Edge.Cuts) (width 0.05))
+  (gr_line (start 155.55 196.5) (end 155.55 199.3) (layer Edge.Cuts) (width 0.05))
+  (gr_arc (start 149.35 17.8) (end 143.15 17.8) (angle -180) (layer Edge.Cuts) (width 0.05))
+  (gr_line (start 155.55 15) (end 283.7 15) (layer Edge.Cuts) (width 0.05))
+  (gr_line (start 143.15 15) (end 143.15 17.8) (layer Edge.Cuts) (width 0.05))
+  (gr_line (start 155.55 15) (end 155.55 17.8) (layer Edge.Cuts) (width 0.05))
+  (dimension 268.7 (width 0.15) (layer Dwgs.User)
+    (gr_text "268,700 mm" (at 149.35 205.8) (layer Dwgs.User)
+      (effects (font (size 1 1) (thickness 0.15)))
+    )
+    (feature1 (pts (xy 15 199.3) (xy 15 205.086421)))
+    (feature2 (pts (xy 283.7 199.3) (xy 283.7 205.086421)))
+    (crossbar (pts (xy 283.7 204.5) (xy 15 204.5)))
+    (arrow1a (pts (xy 15 204.5) (xy 16.126504 203.913579)))
+    (arrow1b (pts (xy 15 204.5) (xy 16.126504 205.086421)))
+    (arrow2a (pts (xy 283.7 204.5) (xy 282.573496 203.913579)))
+    (arrow2b (pts (xy 283.7 204.5) (xy 282.573496 205.086421)))
+  )
+  (dimension 184.3 (width 0.15) (layer Dwgs.User)
+    (gr_text "184,300 mm" (at 289.8 107.15 270) (layer Dwgs.User)
+      (effects (font (size 1 1) (thickness 0.15)))
+    )
+    (feature1 (pts (xy 283.7 199.3) (xy 289.086421 199.3)))
+    (feature2 (pts (xy 283.7 15) (xy 289.086421 15)))
+    (crossbar (pts (xy 288.5 15) (xy 288.5 199.3)))
+    (arrow1a (pts (xy 288.5 199.3) (xy 287.913579 198.173496)))
+    (arrow1b (pts (xy 288.5 199.3) (xy 289.086421 198.173496)))
+    (arrow2a (pts (xy 288.5 15) (xy 287.913579 16.126504)))
+    (arrow2b (pts (xy 288.5 15) (xy 289.086421 16.126504)))
+  )
+  (gr_line (start 283.7 15) (end 283.7 199.3) (layer Edge.Cuts) (width 0.05))
+  (gr_line (start 15 15) (end 15 199.3) (layer Edge.Cuts) (width 0.05))
+  (gr_line (start 15 199.3) (end 143.15 199.3) (layer Edge.Cuts) (width 0.05))
+  (gr_line (start 15 15) (end 143.15 15) (layer Edge.Cuts) (width 0.05))
 )
